File: PLC4UNI_Luis A. G/PLC4UNI_Dev_Board_1.0/ESP32.kicad_sch (KiCad schematic)
At the start: 5 parts, among them U5 ESP32-S3-WR-1

Commit message: Add files via upload
Connections:
- net NPN_MCU is gone; now on net NPN_MCU_1: U5.6 (IO6)
- net PNP_MCU is gone; now on net PNP_MCU_1: U5.18 (IO10)
- net +3.3V: now also R9.1
- net NPN_MCU_1: no longer U5.5 (IO5)
- net NPN_MCU_2: now also U5.5 (IO5); no longer U5.4 (IO4)
- net NPN_MCU_3: now also U5.4 (IO4); no longer U5.15 (IO3)
- net PNP_MCU_1: no longer U5.17 (IO9)
- net PNP_MCU_2: now also U5.17 (IO9); no longer U5.12 (IO8)
- net PNP_MCU_3: now also U5.12 (IO8); no longer U5.7 (IO7)
- net NPN_MC_1 renamed NPN_MC0_1
- new net NPN_MCU_4: U5.15 (IO3)
- new net PNP_MCU_4: U5.7 (IO7)
Other:
- moved on the sheet: C1, R31, R32
