File: PLC4UNI_Luis A. G/PLC4UNI_Dev_Board_1.0/PLC4UNI_Dev_Board_1.0.kicad_sch (KiCad schematic)
At the start: 0 parts

Commit message: Add files via upload
Changed lines of the file:
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@@
 		)
 		(pin "NPN_MC0_1" input
-			(at 107.95 53.34 0)
+			(at 107.95 44.45 0)
 			(effects
 				(font
@@
 		)
 		(pin "NPN_MCO_2" input
-			(at 107.95 55.88 0)
+			(at 107.95 46.99 0)
 			(effects
 				(font
@@
 		)
 		(pin "NPN_MCO_3" input
-			(at 107.95 58.42 0)
+			(at 107.95 49.53 0)
 			(effects
 				(font
@@
 		)
 		(pin "NPN_MCU_1" input
-			(at 107.95 60.96 0)
+			(at 107.95 52.07 0)
 			(effects
 				(font
@@
 		)
 		(pin "NPN_MCU_2" input
-			(at 107.95 63.5 0)
+			(at 107.95 54.61 0)
 			(effects
 				(font
@@
 		)
 		(pin "NPN_MCU_3" input
-			(at 107.95 66.04 0)
+			(at 107.95 57.15 0)
 			(effects
 				(font
@@
 		)
 		(pin "NPN_MCU_4" input
-			(at 107.95 68.58 0)
+			(at 107.95 59.69 0)
 			(effects
 				(font
@@
 		)
 		(pin "UART_OUT" bidirectional
-			(at 38.1 39.37 180)
+			(at 38.1 31.75 180)
 			(effects
 				(font
